File: ATMEGA16U2.sch (KiCad schematic (older format))
At the start: 16 parts, among them U4 ATMEGA16U2-MU, X1 FOXSLF/160-20

Commit message: REV1 Schematic Update
Full schematic revised for compatibility with KiCad v5. All symbols should load from correct libraries, either project associated to a locally included library or to KiCad Default Libraries.

All "rescue" libraries and references cleaned and / or removed.

Manufacturers Part Number "MFP" field name modified to standard "MPN".

Barrel Jack corrected to be center positive. (h/t  Brett who wrote to tell me that).

New BOM CSV file generated.
Parts:
- C10: symbol C -> Device:C; MFP C0805C105K8RACAUTO -> (none); MPN (none) -> C0805C105K8RACAUTO
- C7, C8: symbol C -> Device:C; MFP C0805C200G5GACTU -> (none); MPN (none) -> C0805C200G5GACTU
- C9: symbol C -> Device:C; MFP C0805C104K1RACAUTO -> (none); MPN (none) -> C0805C104K1RACAUTO
- D4: symbol D -> Device:D_Filled; MFP 1N4148W-7-F -> (none); MPN (none) -> 1N4148W-7-F
- D5, D6: symbol LED -> Device:LED_Filled; MFP LG R971-KN-1 -> (none); MPN (none) -> LG R971-KN-1
- ICSP1: symbol CONN_02X03 -> Connector_Generic:Conn_02x03_Odd_Even; MFP M20-9980346 -> (none); MPN (none) -> M20-9980346
- JP2: symbol CONN_02X02 -> Connector_Generic:Conn_02x02_Odd_Even; MFP FOOTPRINT ONLY -> (none); MPN (none) -> FOOTPRINT ONLY
- R10, R11: symbol R -> Device:R; MFP RC0805FR-07510RL -> (none); MPN (none) -> RC0805FR-07510RL
- R7: symbol R -> Device:R; MFP CRCW080510K0JNEA -> (none); MPN (none) -> CRCW080510K0JNEA
- R8: symbol R -> Device:R; MFP ERJ-6GEY0R00V -> (none); MPN (none) -> ERJ-6GEY0R00V
- R9: symbol R -> Device:R; MFP CRCW08051M00FKEA -> (none); MPN (none) -> CRCW08051M00FKEA
- U4: symbol ATMEGA16U2-MU -> MFN_Atmel:ATMEGA16U2-MU; MFP ATMEGA16U2-MU -> (none); MPN (none) -> ATMEGA16U2-MU
- X1: symbol Crystal -> Device:Crystal; MFP FOXSLF/160-20 -> (none); MPN (none) -> FOXSLF/160-20
