File: ATMEGA328P.sch (KiCad schematic (older format))
At the start: 14 parts, among them SW1 RESET_SWITCH, U5 ATMEGA328P, X2 CSTCE16MOV53-R0

Commit message: REV1 Schematic Update
Full schematic revised for compatibility with KiCad v5. All symbols should load from correct libraries, either project associated to a locally included library or to KiCad Default Libraries.

All "rescue" libraries and references cleaned and / or removed.

Manufacturers Part Number "MFP" field name modified to standard "MPN".

Barrel Jack corrected to be center positive. (h/t  Brett who wrote to tell me that).

New BOM CSV file generated.
Parts:
- C11, C14, C15: symbol C -> Device:C; MFP C0805C104K1RACAUTO -> (none); MPN (none) -> C0805C104K1RACAUTO
- D7: symbol D -> Device:D_Filled; MFP 1N4148W-7-F -> (none); MPN (none) -> 1N4148W-7-F
- ICSP2: symbol CONN_02X03 -> Connector_Generic:Conn_02x03_Odd_Even; MFP M20-9980346 -> (none); MPN (none) -> M20-9980346
- R12, R14, R15: symbol R -> Device:R; MFP CRCW08051K00JNEA -> (none); MPN (none) -> CRCW08051K00JNEA
- R13: symbol R -> Device:R; MFP ERJ-6GEY0R00V -> (none); MPN (none) -> ERJ-6GEY0R00V
- R16: symbol R -> Device:R; MFP CRCW080510K0JNEA -> (none); MPN (none) -> CRCW080510K0JNEA
- R17: symbol R -> Device:R; MFP CRCW08051M00FKEA -> (none); MPN (none) -> CRCW08051M00FKEA
- SW1: symbol RESET_SWITCH -> Arduino_Uno_R3_From_Scratch:RESET_SWITCH; MFP EVQ-Q2U02W -> (none); MPN (none) -> EVQ-Q2U02W
- U5: symbol ATMEGA328P-PU -> MFN_Atmel:ATMEGA328P-PU; MFP ATMEGA328P-PU -> (none); MPN (none) -> ATMEGA328P-PU
- X2: symbol CERAMIC_RESONATOR -> Arduino_Uno_R3_From_Scratch:CERAMIC_RESONATOR; MFP CSTCE16M0V53-R0 -> (none); MPN (none) -> CSTCE16M0V53-R0
