File: Arduino_Uno_R3_From_Scratch.sch (KiCad schematic (older format))
At the start: 0 parts

Commit message: REV1 Schematic Update
Full schematic revised for compatibility with KiCad v5. All symbols should load from correct libraries, either project associated to a locally included library or to KiCad Default Libraries.

All "rescue" libraries and references cleaned and / or removed.

Manufacturers Part Number "MFP" field name modified to standard "MPN".

Barrel Jack corrected to be center positive. (h/t  Brett who wrote to tell me that).

New BOM CSV file generated.
Changed lines of the file:
@@
-EESchema Schematic File Version 2
-LIBS:power
-LIBS:device
-LIBS:transistors
-LIBS:conn
-LIBS:linear
-LIBS:regul
-LIBS:74xx
-LIBS:cmos4000
-LIBS:adc-dac
-LIBS:memory
-LIBS:xilinx
-LIBS:microcontrollers
-LIBS:dsp
-LIBS:microchip
-LIBS:analog_switches
-LIBS:motorola
-LIBS:texas
-LIBS:intel
-LIBS:audio
-LIBS:interface
-LIBS:digital-audio
-LIBS:philips
-LIBS:display
-LIBS:cypress
-LIBS:siliconi
-LIBS:opto
-LIBS:atmel
-LIBS:contrib
-LIBS:valves
-LIBS:Arduino_Uno_R3_From_Scratch
-LIBS:MFN_Atmel
-LIBS:MFN_STMicro
-LIBS:Arduino_Uno_R3_From_Scratch-cache
-EELAYER 25 0
+EESchema Schematic File Version 4
+EELAYER 30 0
 EELAYER END
 $Descr A4 11693 8268
@@
 Sheet 1 8
 Title "Arduino UNO R3 Clone"
-Date "8 oct 2015"
-Rev "0"
+Date "2021-08-06"
+Rev "1"
 Comp "Rheingold Heavy"
 Comment1 "Based on the Arduino UNO R3 From arduino.cc"
@@
 	7050 2700 7550 2700
 Wire Wire Line
-	7550 2850 7050 2850
+	7550 2850 7300 2850
 Wire Wire Line
 	7050 3000 7550 3000
@@
 	7300 1750 7300 2850
 Connection ~ 7300 2850
+Wire Wire Line
+	7300 2850 7050 2850
 $EndSCHEMATC
