File: Pin_13_LED.sch (KiCad schematic (older format))
At the start: 3 parts, among them U2 LMV358IDGKR

Commit message: REV1 Schematic Update
Full schematic revised for compatibility with KiCad v5. All symbols should load from correct libraries, either project associated to a locally included library or to KiCad Default Libraries.

All "rescue" libraries and references cleaned and / or removed.

Manufacturers Part Number "MFP" field name modified to standard "MPN".

Barrel Jack corrected to be center positive. (h/t  Brett who wrote to tell me that).

New BOM CSV file generated.
Parts:
- D3: symbol LED -> Device:LED_Filled; MFP LG R971-KN-1 -> (none); MPN (none) -> LG R971-KN-1
- R4: symbol R -> Device:R; MFP RC0805FR-07510RL -> (none); MPN (none) -> RC0805FR-07510RL
- U2: symbol LM358 -> Amplifier_Operational:LMV358; MFP LMV358IDGKR -> (none); MPN (none) -> LMV358IDGKR
Connections:
- net labels removed: 5V_LDO
- wire segments 11 -> 10
Other:
- note added: "Power Pins for U2 LMV358IDGKR (Component C)\nare located with bypass capacitors in the\nVoltage Management schematic."
- moved on the sheet: R4, U2B
Changed lines of the file:
@@
-EESchema Schematic File Version 2
-LIBS:power
-LIBS:device
-LIBS:transistors
-LIBS:conn
-LIBS:linear
-LIBS:regul
-LIBS:74xx
-LIBS:cmos4000
-LIBS:adc-dac
-LIBS:memory
-LIBS:xilinx
-LIBS:microcontrollers
-LIBS:dsp
-LIBS:microchip
-LIBS:analog_switches
-LIBS:motorola
-LIBS:texas
-LIBS:intel
-LIBS:audio
-LIBS:interface
-LIBS:digital-audio
-LIBS:philips
-LIBS:display
-LIBS:cypress
-LIBS:siliconi
-LIBS:opto
-LIBS:atmel
-LIBS:contrib
-LIBS:valves
-LIBS:Arduino_Uno_R3_From_Scratch
-LIBS:MFN_Atmel
-LIBS:MFN_STMicro
-LIBS:Arduino_Uno_R3_From_Scratch-cache
-EELAYER 25 0
+EESchema Schematic File Version 4
+EELAYER 30 0
 EELAYER END
 $Descr A4 11693 8268
@@
 Sheet 4 8
 Title "Arduino UNO R3 Clone"
-Date "8 oct 2015"
-Rev "0"
+Date "2021-08-06"
+Rev "1"
 Comp "Rheingold Heavy"
 Comment1 "Based on the Arduino UNO R3 From arduino.cc"
@@
 Comment4 ""
 $EndDescr
-Text HLabel 4500 3800 0    60   Input ~ 0
+Text HLabel 4550 3875 0    60   Input ~ 0
 SCK
 Wire Wire Line
-	4500 3800 5100 3800
+	5150 4075 5150 4400
 Wire Wire Line
-	5100 4000 4950 4000
+	5150 4400 6150 4400
 Wire Wire Line
-	4950 4000 4950 4450
+	6150 4400 6150 3975
 Wire Wire Line
-	4950 4450 6250 4450
-Wire Wire Line
-	6250 4450 6250 3900
-Wire Wire Line
-	6100 3900 6600 3900
-Wire Wire Line
-	7200 3900 7200 4100
-Wire Wire Line
-	6900 3900 7200 3900
-Connection ~ 6250 3900
-Wire Wire Line
-	5500 3500 5500 3350
+	6650 3975 6950 3975
+Connection ~ 6150 3975
+Wire Notes Line
+	4125 3075 4125 2775
+Wire Notes Line
+	4125 2775 7575 2775
+Wire Notes Line
+	7575 2775 7575 3075
+Text Notes 5275 2725 0    60   ~ 0
+SCK / PIN13 LED Buffer
 $Comp
-L GND #PWR022
-U 1 1 55D7ED46
-P 5500 4700
-F 0 "#PWR022" H 5500 4700 30  0001 C CNN
-F 1 "GND" H 5500 4630 30  0001 C CNN
-F 2 "~" H 5500 4700 60  0000 C CNN
-F 3 "~" H 5500 4700 60  0000 C CNN
-F 4 "ANY" H 5500 4700 60  0001 C CNN "Source"
-F 5 "N" H 5500 4700 60  0001 C CNN "Critical"
-F 6 "~" H 5500 4700 60  0001 C CNN "Notes"
-	1    5500 4700
+L Device:LED_Filled D3
+U 1 1 55D7F0E4
+P 6950 4375
+F 0 "D3" H 6950 4475 50  0000 C CNN
+F 1 "LED" H 6950 4275 50  0000 C CNN
+F 2 "~" H 6950 4375 60  0000 C CNN
+F 3 "http://www.osram-os.com/Graphics/XPic9/00078860_0.pdf" H 6950 4375 60  0001 C CNN
+F 4 "LED CHIPLED 570NM GREEN" H 6950 4375 60  0001 C CNN "Characteristics"
+F 5 "Power On Green LED" H 6950 4375 60  0001 C CNN "Description"
+F 6 "OSRAM Opto" H 6950 4375 60  0001 C CNN "MFN"
+F 7 "SMD_0805" H 6950 4375 60  0001 C CNN "Package ID"
+F 8 "ANY" H 6950 4375 60  0001 C CNN "Source"
+F 9 "N" H 6950 4375 60  0001 C CNN "Critical"
+F 10 "Pin13_LED" H 6950 4375 60  0001 C CNN "Subsystem"
+F 11 "~" H 6950 4375 60  0001 C CNN "Notes"
+F 12 "LG R971-KN-1" H 6950 4375 50  0001 C CNN "MPN"
+	1    6950 4375
+	0    -1   -1   0
+$EndComp
+$Comp
+L Device:R R4
+U 1 1 55D7F236
+P 6500 3975
+F 0 "R4" V 6580 3975 40  0000 C CNN
+F 1 "510" V 6500 3975 40  0000 C CNN
+F 2 "~" V 6430 3975 30  0000 C CNN
+F 3 "http://www.yageo.com/pdf/Pu-RC0805_51_PbFree_L_2.pdf" H 6500 3975 30  0001 C CNN
+F 4 "RESISTOR, METAL GLAZE/THICK FILM, 0.125W, 1%, 100ppm, 510ohm, SURFACE MOUNT, 0805" H 6500 3975 60  0001 C CNN "Characteristics"
+F 5 "Power On LED Resistor" H 6500 3975 60  0001 C CNN "Description"
+F 6 "Yageo" H 6500 3975 60  0001 C CNN "MFN"
+F 7 "SMD_0805" H 6500 3975 60  0001 C CNN "Package ID"
+F 8 "ANY" H 6500 3975 60  0001 C CNN "Source"
+F 9 "N" H 6500 3975 60  0001 C CNN "Critical"
+F 10 "Pin13_LED" H 6500 3975 60  0001 C CNN "Subsystem"
+F 11 "~" H 6500 3975 60  0001 C CNN "Notes"
+F 12 "RC0805FR-07510RL" H 6500 3975 50  0001 C CNN "MPN"
+	1    6500 3975
+	0    -1   -1   0
+$EndComp
+$Comp
+L power:GND #PWR024
+U 1 1 561FF2A3
+P 6950 4775
+F 0 "#PWR024" H 6950 4775 30  0001 C CNN
+F 1 "GND" H 6950 4705 30  0001 C CNN
+F 2 "~" H 6950 4775 60  0000 C CNN
+F 3 "~" H 6950 4775 60  0000 C CNN
+F 4 "ANY" H 6950 4775 60  0001 C CNN "Source"
+F 5 "N" H 6950 4775 60  0001 C CNN "Critical"
+F 6 "~" H 6950 4775 60  0001 C CNN "Notes"
+	1    6950 4775
 	1    0    0    -1
 $EndComp
 Wire Wire Line
-	5500 4300 5500 4700
-Wire Notes Line
-	3950 3000 3950 2700
-Wire Notes Line
-	3950 2700 7400 2700
-Wire Notes Line
-	7400 2700 7400 3000
-Wire Wire Line
-	7200 4500 7200 4700
-Text Notes 5100 2650 0    60   ~ 0
-SCK / PIN13 LED Buffer
+	6150 3975 6350 3975
 $Comp
-L LM358 U2
+L Amplifier_Operational:LMV358 U2
 U 2 1 55D7ED66
-P 5600 3900
-F 0 "U2" H 5550 4100 60  0000 L CNN
-F 1 "LMV358IDGKR" H 5550 3650 60  0000 L CNN
-F 2 "~" H 5600 3900 60  0000 C CNN
-F 3 "http://www.ti.com/lit/ds/symlink/lmv358.pdf" H 5600 3900 60  0001 C CNN
-F 4 "DUAL OP-AMP, 7000uV OFFSET-MAX, 1MHz BAND WIDTH" H 5600 3900 60  0001 C CNN "Characteristics"
-F 5 "Comparator Op-amp" H 5600 3900 60  0001 C CNN "Description"
-F 6 "Texas Instruments" H 5600 3900 60  0001 C CNN "MFN"
-F 7 "LMV358IDGKR" H 5600 3900 60  0001 C CNN "MFP"
-F 8 "VSSOP8" H 5600 3900 60  0001 C CNN "Package ID"
-F 9 "ANY" H 5600 3900 60  0001 C CNN "Source"
-F 10 "N" H 5600 3900 60  0001 C CNN "Critical"
-F 11 "Pin13_LED" H 5600 3900 60  0001 C CNN "Subsystem"
-F 12 "~" H 5600 3900 60  0001 C CNN "Notes"
-	2    5600 3900
+P 5650 3975
+F 0 "U2" H 5600 4175 60  0000 L CNN
+F 1 "LMV358IDGKR" H 5350 3700 60  0000 L CNN
+F 2 "~" H 5650 3975 60  0000 C CNN
+F 3 "http://www.ti.com/lit/ds/symlink/lmv358.pdf" H 5650 3975 60  0001 C CNN
+F 4 "DUAL OP-AMP, 7000uV OFFSET-MAX, 1MHz BAND WIDTH" H 5650 3975 60  0001 C CNN "Characteristics"
+F 5 "Comparator Op-amp" H 5650 3975 60  0001 C CNN "Description"
+F 6 "Texas Instruments" H 5650 3975 60  0001 C CNN "MFN"
+F 7 "VSSOP8" H 5650 3975 60  0001 C CNN "Package ID"
+F 8 "ANY" H 5650 3975 60  0001 C CNN "Source"
+F 9 "N" H 5650 3975 60  0001 C CNN "Critical"
+F 10 "Pin13_LED" H 5650 3975 60  0001 C CNN "Subsystem"
+F 11 "~" H 5650 3975 60  0001 C CNN "Notes"
+F 12 "LMV358IDGKR" H 5650 3975 50  0001 C CNN "MPN"
+	2    5650 3975
 	1    0    0    -1
 $EndComp
-$Comp
-L LED D3
-U 1 1 55D7F0E4
-P 7200 4300
-F 0 "D3" H 7200 4400 50  0000 C CNN
-F 1 "LED" H 7200 4200 50  0000 C CNN
-F 2 "~" H 7200 4300 60  0000 C CNN
-F 3 "http://www.osram-os.com/Graphics/XPic9/00078860_0.pdf" H 7200 4300 60  0001 C CNN
-F 4 "LED CHIPLED 570NM GREEN" H 7200 4300 60  0001 C CNN "Characteristics"
-F 5 "Power On Green LED" H 7200 4300 60  0001 C CNN "Description"
-F 6 "OSRAM Opto" H 7200 4300 60  0001 C CNN "MFN"
-F 7 "LG R971-KN-1" H 7200 4300 60  0001 C CNN "MFP"
-F 8 "SMD_0805" H 7200 4300 60  0001 C CNN "Package ID"
-F 9 "ANY" H 7200 4300 60  0001 C CNN "Source"
-F 10 "N" H 7200 4300 60  0001 C CNN "Critical"
-F 11 "Pin13_LED" H 7200 4300 60  0001 C CNN "Subsystem"
-F 12 "~" H 7200 4300 60  0001 C CNN "Notes"
-	1    7200 4300
-	0    -1   -1   0
-$EndComp
-$Comp
-L R R4
-U 1 1 55D7F236
-P 6750 3900
-F 0 "R4" V 6830 3900 40  0000 C CNN
-F 1 "510" V 6757 3901 40  0000 C CNN
-F 2 "~" V 6680 3900 30  0000 C CNN
-F 3 "http://www.yageo.com/pdf/Pu-RC0805_51_PbFree_L_2.pdf" H 6750 3900 30  0001 C CNN
-F 4 "RESISTOR, METAL GLAZE/THICK FILM, 0.125W, 1%, 100ppm, 510ohm, SURFACE MOUNT, 0805" H 6750 3900 60  0001 C CNN "Characteristics"
-F 5 "Power On LED Resistor" H 6750 3900 60  0001 C CNN "Description"
-F 6 "Yageo" H 6750 3900 60  0001 C CNN "MFN"
-F 7 "RC0805FR-07510RL" H 6750 3900 60  0001 C CNN "MFP"
-F 8 "SMD_0805" H 6750 3900 60  0001 C CNN "Package ID"
-F 9 "ANY" H 6750 3900 60  0001 C CNN "Source"
-F 10 "N" H 6750 3900 60  0001 C CNN "Critical"
-F 11 "Pin13_LED" H 6750 3900 60  0001 C CNN "Subsystem"
-F 12 "~" H 6750 3900 60  0001 C CNN "Notes"
-	1    6750 3900
-	0    -1   -1   0
-$EndComp
-$Comp
-L 5V_LDO #PWR023
-U 1 1 55E95C9F
-P 5500 3350
-F 0 "#PWR023" H 5500 3440 20  0001 C CNN
-F 1 "5V_LDO" H 5500 3470 30  0000 C CNN
-F 2 "~" H 5500 3350 60  0000 C CNN
-F 3 "~" H 5500 3350 60  0000 C CNN
-	1    5500 3350
-	1    0    0    -1
-$EndComp
-$Comp
-L GND #PWR024
-U 1 1 561FF2A3
-P 7200 4700
-F 0 "#PWR024" H 7200 4700 30  0001 C CNN
-F 1 "GND" H 7200 4630 30  0001 C CNN
-F 2 "~" H 7200 4700 60  0000 C CNN
-F 3 "~" H 7200 4700 60  0000 C CNN
-F 4 "ANY" H 7200 4700 60  0001 C CNN "Source"
-F 5 "N" H 7200 4700 60  0001 C CNN "Critical"
-F 6 "~" H 7200 4700 60  0001 C CNN "Notes"
-	1    7200 4700
-	1    0    0    -1
-$EndComp
+Wire Wire Line
+	5950 3975 6150 3975
+Wire Wire Line
+	5150 4075 5350 4075
+Wire Wire Line
+	4550 3875 5350 3875
+Wire Wire Line
+	6950 4525 6950 4775
+Wire Wire Line
+	6950 3975 6950 4225
+Text Notes 4400 5350 2    50   ~ 0
+Power Pins for U2 LMV358IDGKR (Component C)\nare located with bypass capacitors in the\nVoltage Management schematic.
+Wire Notes Line
+	4450 5075 4450 5375
+Wire Notes Line
+	4450 5225 5625 5225
+Wire Notes Line
+	5625 5225 5625 4500
 $EndSCHEMATC
