File: USB_Interface.sch (KiCad schematic (older format))
At the start: 7 parts, among them J1 USB_TYPE_B

Commit message: REV1 Schematic Update
Full schematic revised for compatibility with KiCad v5. All symbols should load from correct libraries, either project associated to a locally included library or to KiCad Default Libraries.

All "rescue" libraries and references cleaned and / or removed.

Manufacturers Part Number "MFP" field name modified to standard "MPN".

Barrel Jack corrected to be center positive. (h/t  Brett who wrote to tell me that).

New BOM CSV file generated.
Parts:
- FB1: symbol FILTER -> Device:FerriteBead; MFP BLM21PG221SN1D -> (none); MPN (none) -> BLM21PG221SN1D
- J1: symbol USB_TYPE_B -> Arduino_Uno_R3_From_Scratch:USB_TYPE_B; MFP 292304-1 -> (none); MPN (none) -> 292304-1
- MF-MSMF050-2: symbol THERMISTOR -> Device:Thermistor; MFP MF-MSMF050-2 -> (none); MPN (none) -> MF-MSMF050-2
- R5, R6: symbol R -> Device:R; MFP RC0805JR-0722RL -> (none); MPN (none) -> RC0805JR-0722RL
- VR1, VR2: symbol VR -> Device:Thermistor; MFP CG0603MLC-05E -> (none); MPN (none) -> CG0603MLC-05E
Connections:
- net USB_GND: now also FB1.2; no longer FB1.1
- net at J1.5 (Shield_1), J1.6 (Shield_2), VR1.2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: now also FB1.1; no longer FB1.2
Other:
- note added: "PIN 4 GND will throw an ERC error due to\nthe pin being separated from GND by a 0R\nresistor in the ATMEGA16U2 schematic.\nThis error is accepted."
- moved on the sheet: J1, R5, R6, VR1, VR2
