File: Voltage_Regulator.sch (KiCad schematic (older format))
At the start: 8 parts, among them CON1 BARREL_JACK, U1 LD1117S50TR

Commit message: REV1 Schematic Update
Full schematic revised for compatibility with KiCad v5. All symbols should load from correct libraries, either project associated to a locally included library or to KiCad Default Libraries.

All "rescue" libraries and references cleaned and / or removed.

Manufacturers Part Number "MFP" field name modified to standard "MPN".

Barrel Jack corrected to be center positive. (h/t  Brett who wrote to tell me that).

New BOM CSV file generated.
Parts:
- C1, C2: symbol CP -> Device:C_Polarized; MFP MAL215371479E3 -> (none); MPN (none) -> MAL215371479E3
- C3: symbol C -> Device:C; MFP C0805C104K1RACAUTO -> (none); MPN (none) -> C0805C104K1RACAUTO
- CON1: symbol BARREL_JACK -> Arduino_Uno_R3_From_Scratch:BARREL_JACK; MFP 694106106102 -> (none); MPN (none) -> 694106106102
- D1: symbol D -> Device:D_Filled; MFP MRA4007T3G -> (none); MPN (none) -> MRA4007T3G
- D2: symbol LED -> Device:LED_Filled; MFP LG R971-KN-1 -> (none); MPN (none) -> LG R971-KN-1
- R1: symbol R -> Device:R; MFP RC0805FR-07510RL -> (none); MPN (none) -> RC0805FR-07510RL
- U1: symbol LD1117S50TR -> MFN_STMicro:LD1117S50TR; MFP LD1117S50TR -> (none); MPN (none) -> LD1117S50TR
Connections:
- net GND: now also CON1.2, CON1.3; no longer CON1.1
- new net: CON1.1, D1.2 (A)
Other:
- note added: "Power Flags for ERC"
- moved on the sheet: C3, CON1, R1, U1
