File: voltage_management.sch (KiCad schematic (older format))
At the start: 8 parts, among them Q1 FDN340P, U2 LMV358IDGKR, U3 LP2985-33DBVR

Commit message: REV1 Schematic Update
Full schematic revised for compatibility with KiCad v5. All symbols should load from correct libraries, either project associated to a locally included library or to KiCad Default Libraries.

All "rescue" libraries and references cleaned and / or removed.

Manufacturers Part Number "MFP" field name modified to standard "MPN".

Barrel Jack corrected to be center positive. (h/t  Brett who wrote to tell me that).

New BOM CSV file generated.
Parts:
- added unit 3 of U2
- C4: symbol C -> Device:C; MFP C0805C104K1RACAUTO -> (none); MPN (none) -> C0805C104K1RACAUTO
- C5: symbol C -> Device:C; MFP C0805C105K8RACAUTO -> (none); MPN (none) -> C0805C105K8RACAUTO
- C6: symbol C -> Device:C; MFP C2012X7R1C225K125AB -> (none); MPN (none) -> C2012X7R1C225K125AB
- Q1: symbol Q_PMOS_GSD -> Device:Q_PMOS_GSD; MFP FDN340P -> (none); MPN (none) -> FDN340P
- R2, R3: symbol R -> Device:R; MFP CRCW080510K0JNEA -> (none); MPN (none) -> CRCW080510K0JNEA
- U2: symbol LM358 -> Amplifier_Operational:LMV358; MFP LMV358IDGKR -> (none); MPN (none) -> LMV358IDGKR
- U3: symbol LP2985LV -> Regulator_Linear:LP2985-3.3; MFP LP2985-33DBVR -> (none); MPN (none) -> LP2985-33DBVR
Connections:
- wire segments 25 -> 31
Other:
- moved on the sheet: C4, C5, C6, R2, R3, U2A
